File: pcb_main_r2/mintypcb.kicad_sch (KiCad schematic)
At the start: 123 parts, among them J101 USB C 6 pin, J102 S2B-PH-SM4-TB, J103 2005280080, Q101 3415, Q102 3415, Q103 BSS138, SW101 SKQGABE010, SW102 SKRRAAE010, SW103 SKQGABE010, SW104 SKRRAAE010, SW105 SKQGABE010, SW106 SKRRAAE010, SW107 see note 1, SW108 SKRRAAE010, SW109 see note 1, SW110 SKRRAAE010, SW111 see note 1, SW112 SKRRAAE010, SW113 see note 1, SW114 SKRRAAE010, SW115 SKQGABE010, SW116 SKRRAAE010, U101 LMV393, U102 MCP73833T-FCI/MF, U103 PAM2401, U104 MAX98357A

Commit message: production 3D and PCB files
Parts:
- added J106: Conn_02x15_Odd_Even, Custom:pi_tin_pi_simulator, symbol Connector_Generic:Conn_02x15_Odd_Even
- added J107: Conn_02x15_Odd_Even, Custom:pi_tin_pi_simulator_lands, symbol Connector_Generic:Conn_02x15_Odd_Even
- added J108: Conn_02x15_Odd_Even, Custom:pi_tin_pi_simulator_tp, symbol Connector_Generic:Conn_02x15_Odd_Even
- A101: footprint Custom:RASPBERRYPI-ZERO_RPI-ZERO -> Custom:RASPBERRYPI-ZERO_RPI-ZERO_pi_tin; Availability Not in stock -> (none); Check_prices https://www.snapeda.com/parts/RASPBERRYPI-ZERO/Raspberry+Pi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 -> (none); Description_1 Official Raspberry Pi Zero Case -> (none); MANUFACTURER Raspberry -> (none); MF Raspberry Pi -> (none); MPN (Alternate) (none) -> SC1176; Package None -> (none); Price None -> (none); Rev. 1 MPN SC1176 -> (none); STANDARD MAnufactutrer Recommendations -> (none); SnapEDA_Link https://www.snapeda.com/parts/RASPBERRYPI-ZERO/Raspberry+Pi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 -> (none); now left out of the parts list
- C101, C102, C105: LCSC (none) -> C87996; MPN (none) -> CL31B226KPHNNNE; Rev. 1 MPN CL31B226KPHNNNE -> (none)
- C103, C104, C108: LCSC (none) -> C32635; MPN (none) -> CL21B106KPQNNNE; Rev. 1 MPN CL21B106KPQNNNE -> (none)
- C106, C109, C112: LCSC (none) -> C14663; MPN (none) -> CC0603KRX7R9BB104; MPN (Alternate) (none) -> CL10B104KB8NNWC; Rev. 1 MPN CL10B104KB8NNWC -> (none)
- C110, C111: MPN (Alternate) (none) -> CL10C221JB8NNNC; Rev. 1 MPN CL10C221JB8NNNC -> (none)
- D101: LCSC (none) -> C64888; MPN (none) -> DSK110 K110; MPN (Alternate) (none) -> DSK110; Rev. 1 MPN DSK110 -> (none)
- D102: LCSC (none) -> C157740; MPN (none) -> LTST-C190KFKT; MPN (Alternate) (none) -> B1911UD--20D001014U1930; Rev. 1 MPN B1911UD--20D001014U1930 -> (none)
- D104: LCSC (none) -> C364559; MPN (none) -> LTST-C190TGKT; MPN (Alternate) (none) -> B1911NG--20D000214U1930; Rev. 1 MPN B1911NG--20D000214U1930 -> (none)
- D105, D106, D107: LCSC (none) -> C124205; MPN (none) -> BAT54WS-7-F; Rev. 1 MPN BAT54WS-7-F -> (none)
- F101: LCSC (none) -> C151139; MPN (none) -> 0467001.NRHF; MPN (Alternate) (none) -> FMC16102WHTP; Rev. 1 MPN FMC16102WHTP -> (none)
- FB103, FB104: MPN (Alternate) (none) -> BLM18AG121SZ1D; Rev. 1 MPN BLM18AG121SZ1D -> (none)
- J101: footprint Custom:USB_C_Receptacle_GT_USB_7002F -> Custom:USB_C_Receptacle_6PIN_generic; LCSC (none) -> C668623; MPN (none) -> TYPE-C 6P(073); MPN (Alternate) (none) -> USB4125-GF-A; Rev. 1 MPN USB4125-GF-A -> (none)
- J102: LCSC (none) -> C295747; MPN (none) -> S2B-PH-SM4-TB; Rev. 1 MPN S2B-PH-SM4-TB -> (none)
- J103: value 2005280080 -> FPC09-Q1.0-8; footprint Custom:Molex_200528-0080_1x08-1MP_P1.00mm_Horizontal -> Custom:XYECONN_FPC09-Q1.0-8AH2.0; LCSC (none) -> C19269923; MPN (none) -> FPC09-Q1.0-8AH2.0; Rev. 1 MPN 2005280080 -> (none)
- L101: LCSC (none) -> C5832385; MPN (none) -> FTC322512S2R2MBCA; MPN (Alternate) (none) -> WIP322512A-2R2MLDG; Rev. 1 MPN WIP322512A-2R2MLDG -> (none)
- LS101: MPN (Alternate) (none) -> CMS-151125-076S-67; Rev. 1 MPN CMS-151125-076S-67 -> (none); now left out of the parts list
- Q101, Q102: LCSC (none) -> C337518; MPN (none) -> 3415A; MPN (Alternate) (none) -> GSFC3415C; Rev. 1 MPN GSFC3415C -> (none)
- Q103: LCSC (none) -> C24553; MPN (none) -> BSS138W-7-F; MPN (Alternate) (none) -> BSS138BKW-TP; Rev. 1 MPN BSS138BKW-TP -> (none)
- R101, R111, R121: LCSC (none) -> C25804; MPN (none) -> 0603WAF1002T5E
- R102, TP101, TP102, TP103, TP104, TP105, TP106, TP107, TP108, TP109, TP110, TP111, TP112, TP113, TP114, TP115, TP116, TP117, TP118, TP119, TP120, TP121, TP122, TP123, TP124, TP125, TP126, TP127, TP128, TP129, TP130, TP131: now left out of the parts list
- R104, R128: LCSC (none) -> C23345; MPN (none) -> 0603WAF220JT5E
- R105, R109, R110, R114, R120: LCSC (none) -> C22846; MPN (none) -> 0603WAF1691T5E
- R106, R112, R113, R115, R122, R125, R127, R129: LCSC (none) -> C25803; MPN (none) -> 0603WAF1003T5E
- R107: LCSC (none) -> C23184; MPN (none) -> 0603WAF4992T5E
- R108, R126: LCSC (none) -> C23240; MPN (none) -> 0603WAF7503T5E
- R116, R117, R123, R124: LCSC (none) -> C23186; MPN (none) -> 0603WAF5101T5E
- R119: LCSC (none) -> C23231; MPN (none) -> 0603WAF6802T5E
- SW101, SW103, SW105, SW115: LCSC (none) -> C115351; MPN (none) -> SKQGABE010; MPN (Alternate) (none) -> PTS526SM15SMTR2 LFS; Rev. 1 MPN SKQGABE010 -> (none)
- SW102, SW104, SW106, SW108, SW110, SW112, SW114, SW116: footprint Custom:SW_PTS526_or_SKRR -> Custom:SW_SKRR; LCSC (none) -> C97437; MPN (none) -> SKRRAAE010; Rev. 1 MPN SKRRAAE010 -> (none)
- SW107, SW109, SW111, SW113: footprint Custom:SW_TL3336AF160Q_or_PTS645 -> Custom:SW_TL3336AF160Q_or_PTS645_paste1; LCSC (none) -> C231324; MPN (none) -> B3FS-1010P; MPN (Alternate) (none) -> TL3336AF160Q; Rev. 1 MPN TL3336AF160Q -> (none)
- U101: LCSC (none) -> C460091; MPN (none) -> LMV393M8-13; MPN (Alternate) (none) -> LMV393X-VS1R; Rev. 1 MPN LMV393X-VS1R -> (none)
- U102: LCSC (none) -> C511337; MPN (none) -> MCP73833T-FCI/MF; Rev. 1 MPN MCP73833T-FCI/MF -> (none)
- U103: value PAM2401 -> PAM2401SCADJ; LCSC (none) -> C508238; MPN (none) -> PAM2401SCADJ; Rev. 1 MPN PAM2401SCADJ -> (none)
- U104: LCSC (none) -> C910544; MPN (none) -> MAX98357AETE+T; Rev. 1 MPN MAX98357AETE+T -> (none)
Connections:
- new net: J107.1 (Pin_1), J108.1 (Pin_1)
- new net: J107.10 (Pin_10), J108.10 (Pin_10)
- new net: J107.11 (Pin_11), J108.11 (Pin_11)
- new net: J107.12 (Pin_12), J108.12 (Pin_12)
- new net: J107.13 (Pin_13), J108.13 (Pin_13)
- new net: J107.14 (Pin_14), J108.14 (Pin_14)
- new net: J107.15 (Pin_15), J108.15 (Pin_15)
- new net: J107.16 (Pin_16), J108.16 (Pin_16)
- new net: J107.17 (Pin_17), J108.17 (Pin_17)
- new net: J107.18 (Pin_18), J108.18 (Pin_18)
- new net: J107.19 (Pin_19), J108.19 (Pin_19)
- new net: J107.2 (Pin_2), J108.2 (Pin_2)
- new net: J107.20 (Pin_20), J108.20 (Pin_20)
- new net: J107.21 (Pin_21), J108.21 (Pin_21)
- new net: J107.22 (Pin_22), J108.22 (Pin_22)
- new net: J107.23 (Pin_23), J108.23 (Pin_23)
- new net: J107.24 (Pin_24), J108.24 (Pin_24)
- new net: J107.25 (Pin_25), J108.25 (Pin_25)
- new net: J107.26 (Pin_26), J108.26 (Pin_26)
- new net: J107.27 (Pin_27), J108.27 (Pin_27)
- new net: J107.28 (Pin_28), J108.28 (Pin_28)
- new net: J107.29 (Pin_29), J108.29 (Pin_29)
- new net: J107.3 (Pin_3), J108.3 (Pin_3)
- new net: J107.30 (Pin_30), J108.30 (Pin_30)
- new net: J107.4 (Pin_4), J108.4 (Pin_4)
- new net: J107.5 (Pin_5), J108.5 (Pin_5)
- new net: J107.6 (Pin_6), J108.6 (Pin_6)
- new net: J107.7 (Pin_7), J108.7 (Pin_7)
- new net: J107.8 (Pin_8), J108.8 (Pin_8)
- new net: J107.9 (Pin_9), J108.9 (Pin_9)
Other:
- note added: "note 1: for mint tin case use B3FS-1010P or PTS645SM43SMTR92 LFS (6mm x 4.3mm SMT vertical tactile) for 3d printed case use TL3336AF160Q (6mm x 4mm SMD right angle tactile) power sequencing: startup: SW101 turns BATT switch Q102 on through Q103 (BATT_SW_EN) R111 latches Q102 on through Q103 normal operation: SHUTDOWN_PI (active high) is pulled up by ~50K internal pullup LOW_BATT is LOW, causing S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"
- note removed: "note 1: for mint tin case use PTS645SM43SMTR92 LFS (6mm x 4.3mm SMT vertical tactile) for 3d printed case use TL3336AF160Q (6mm x 4mm SMD right angle tactile) power sequencing: startup: SW101 turns BATT switch Q102 on through Q103 (BATT_SW_EN) R111 latches Q102 on through Q103 normal operation: SHUTDOWN_PI (active high) is pulled up by ~50K internal pullup LOW_BATT is LOW, causing SHUTDOWN_PI to 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"
